File: pcb.kicad_sch (KiCad schematic)
At the start: 27 parts, among them J1 Conn_02x20_Odd_Even, J2 USB_C_Receptacle_PowerOnly_6P, J3 Conn_01x05_Socket, J4 Conn_01x05_Socket, J5 Conn_01x04, Q1 2N7002K, Q2 2N7002

Commit message: Schaltplan sensorpcb hinzugefügt und Schaltplan pcb, bom bearbeitet
Parts:
- added D7: LED_365, LED_SMD:LED_PLCC_2835, symbol Device:LED
- added R10, R11, R12, R13: 51R, Resistor_SMD:R_0603_1608Metric, symbol Device:R
- added R14, R16, R7, R9: 56R, Resistor_SMD:R_0603_1608Metric, symbol Device:R
- added R15, R8: 43R, Resistor_SMD:R_0603_1608Metric, symbol Device:R
- added R17, R18, R19, R20, R21, R22, R23, R24, R25: 68R, Resistor_SMD:R_0603_1608Metric, symbol Device:R
- added R3, R4, R5, R6: 0R, Resistor_SMD:R_0805_2012Metric_Pad1.20x1.40mm_HandSolder, symbol Device:R
- D1: renamed from D4; value LED -> LED_405; footprint (none) -> LED_SMD:LED_PLCC-2_3.4x3.0mm_KA
- D10: renamed from D18; value LED -> LED_405; footprint (none) -> LED_SMD:LED_PLCC-2_3.4x3.0mm_KA
- D11: value LED -> LED_w; footprint (none) -> LED_SMD:LED_PLCC_2835; MPN (none) -> EAPL2835WA5
- D12: renamed from D10; value LED -> LED_w; footprint (none) -> LED_SMD:LED_PLCC_2835; MPN (none) -> EAPL2835WA5
- D13: renamed from D9; value LED -> LED_w; footprint (none) -> LED_SMD:LED_PLCC_2835; MPN (none) -> EAPL2835WA5
- D14: renamed from D7; value LED -> LED_w; footprint (none) -> LED_SMD:LED_PLCC_2835; MPN (none) -> EAPL2835WA5
- D15: renamed from D6; value LED -> LED_w; footprint (none) -> LED_SMD:LED_PLCC_2835; MPN (none) -> EAPL2835WA5
- D16: renamed from D5; value LED -> LED_w; footprint (none) -> LED_SMD:LED_PLCC_2835; MPN (none) -> EAPL2835WA5
- D17: renamed from D3; value LED -> LED_w; footprint (none) -> LED_SMD:LED_PLCC_2835; MPN (none) -> EAPL2835WA5
- D18: renamed from D2; value LED -> LED_w; footprint (none) -> LED_SMD:LED_PLCC_2835; MPN (none) -> EAPL2835WA5
- D19: renamed from D1; value LED -> LED_w; footprint (none) -> LED_SMD:LED_PLCC_2835; MPN (none) -> EAPL2835WA5
- D2: renamed from D8; value LED -> LED_blue; footprint (none) -> LED_SMD:LED_PLCC-2_3.4x3.0mm_AK
- D3: renamed from D12; value LED -> LED_405; footprint (none) -> LED_SMD:LED_PLCC-2_3.4x3.0mm_KA
- D4: renamed from D13; value LED -> LED_365; footprint (none) -> LED_SMD:LED_PLCC_2835
- D5: renamed from D14; value LED -> LED_365; footprint (none) -> LED_SMD:LED_PLCC_2835
- D6: renamed from D15; value LED -> LED_365; footprint (none) -> LED_SMD:LED_PLCC_2835
- D8: renamed from D16; value LED -> LED_405; footprint (none) -> LED_SMD:LED_PLCC-2_3.4x3.0mm_KA
- D9: renamed from D17; value LED -> LED_blue; footprint (none) -> LED_SMD:LED_PLCC-2_3.4x3.0mm_AK
- J1: renamed from J2; footprint (none) -> Connector_USB:USB_C_Receptacle_JAE_DX07S024WJ3R400
- J2: renamed from J1; footprint (none) -> Connector_PinSocket_2.54mm:PinSocket_2x20_P2.54mm_Vertical
- J3: renamed from J5; footprint (none) -> Connector_PinSocket_2.54mm:PinSocket_1x04_P2.54mm_Vertical
- J4: renamed from J3; footprint (none) -> Connector_PinSocket_2.54mm:PinSocket_1x05_P2.54mm_Vertical
- J5: renamed from J4; footprint (none) -> Connector_PinSocket_2.54mm:PinSocket_1x05_P2.54mm_Vertical
- R1, R2: value R -> 5k1; footprint (none) -> Resistor_SMD:R_0603_1608Metric
- renumbered Q2 to Q1, Q1 to Q2
Connections:
- net +5V: now also R10.2, R11.2, R12.2, R13.2, R14.2, R15.2, R16.2, R17.2, R18.2, R19.2, R20.2, R21.2, R22.2, R23.2, R24.2, R25.2, R7.2, R8.2, R9.2; no longer R1.1, R2.1
- net GND: now also R1.1, R2.1
- net RX: now also R3.1, R5.1; no longer J4.1 (Pin_1)
- net TX: now also R4.1, R6.1; no longer J4.2 (Pin_2)
- net at D1.1 (K), D10.1 (K), D2.1 (K)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: now also D7.1 (K)
- net at J1.A5 (CC1): now also R2.2
- net at J1.B5 (CC2): now also R1.2
- new net: D12.2 (A), R18.1
- new net: D3.2 (A), R9.1
- new net: D11.2 (A), R17.1
- new net: D5.2 (A), R11.1
- new net: J4.1 (Pin_1), R3.2, R4.2
- new net: D19.2 (A), R25.1
- new net: D9.2 (A), R15.1
- new net: D14.2 (A), R20.1
- new net: D10.2 (A), R16.1
- new net: D4.2 (A), R10.1
- new net: J4.2 (Pin_2), R5.2, R6.2
- new net: D2.2 (A), R8.1
- new net: D7.2 (A), R13.1
- new net: D17.2 (A), R23.1
- new net: D13.2 (A), R19.1
- new net: D16.2 (A), R22.1
- new net: D15.2 (A), R21.1
- new net: D8.2 (A), R14.1
- new net: D1.2 (A), R7.1
- new net: D6.2 (A), R12.1
- new net: D18.2 (A), R24.1
Other:
- moved on the sheet: D1, D10, D2, D3, D4, D5, D6, D8, D9, J2, J3, J4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

Commit message: Update Schaltplan
Parts:
- removed J3: Conn_01x04, Connector_PinSocket_2.54mm:PinSocket_1x04_P2.54mm_Vertical, symbol Connector_Generic:Conn_01x04
- removed Q1: 2N7002, Package_TO_SOT_SMD:SOT-23, symbol Transistor_FET:2N7002
- removed Q2: 2N7002K, Package_TO_SOT_SMD:SOT-23, symbol Transistor_FET:2N7002K
- added Q1, Q2: DMG1012T, Package_TO_SOT_SMD:SOT-523, symbol Transistor_FET:DMG1012T
- added R3, R4: 4k7, Resistor_SMD:R_0805_2012Metric_Pad1.20x1.40mm_HandSolder, symbol Device:R
- added U1: BME280, Package_LGA:Bosch_LGA-8_2.5x2.5mm_P0.65mm_ClockwisePinNumbering, symbol Sensor:BME280
- J1: footprint Connector_USB:USB_C_Receptacle_JAE_DX07S024WJ3R400 -> Connector_USB:USB_C_Receptacle_Amphenol_12401610E4-2A
- renumbered J4 to J3, J5 to J4, R8 to R10, R9 to R11, R10 to R12, R11 to R13, R12 to R14, R13 to R15, R14 to R16, R15 to R17, R16 to R18, R17 to R19, R18 to R20, R19 to R21, R20 to R22, R21 to R23, R22 to R24, R23 to R25, R24 to R26, R25 to R27, R3 to R5, R4 to R6, R5 to R7, R6 to R8, R7 to R9
Connections:
- net +3.3V: now also J4.3 (Pin_3), R3.1, R4.1, U1.2 (CSB), U1.6 (VDDIO), U1.8 (VDD)
- net +5V: no longer J4.4 (Pin_4)
- net GND: now also Q1.2 (S), Q2.2 (S), U1.1 (GND), U1.5 (SDO), U1.7 (GND)
- net SCL: now also R4.2, U1.4 (SCK)
- net SDA: now also R3.2, U1.3 (SDI)
- net led_uv_enable: now also Q1.1 (G)
- net led_white_enable: now also Q2.1 (G)
- net at D11.1 (K), D12.1 (K), D13.1 (K)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: now also Q2.3 (D)
- net at D1.1 (K), D10.1 (K), D2.1 (K)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: now also Q1.3 (D)
